File: inkplateclone.sch (KiCad schematic (older format))
At the start: 42 parts, among them J2 Conn_01x16_Male, U1 TPS65186, U2 ED097OC1, U3 MCP23017_SO

Commit message: ED060SC7 as a symbol now
Parts:
- C20, C21, C22: value 100n -> 100nF
Changed lines of the file:
@@
 P 10950 1300
 F 0 "C20" H 10835 1254 50  0000 R CNN
-F 1 "100n" H 10835 1345 50  0000 R CNN
+F 1 "100nF" H 10835 1345 50  0000 R CNN
 F 2 "Capacitor_SMD:C_0805_2012Metric" H 10988 1150 50  0001 C CNN
 F 3 "~" H 10950 1300 50  0001 C CNN
@@
 P 11400 1300
 F 0 "C21" H 11285 1254 50  0000 R CNN
-F 1 "100n" H 11285 1345 50  0000 R CNN
+F 1 "100nF" H 11285 1345 50  0000 R CNN
 F 2 "Capacitor_SMD:C_0805_2012Metric" H 11438 1150 50  0001 C CNN
 F 3 "~" H 11400 1300 50  0001 C CNN
@@
 P 8600 5700
 F 0 "C22" H 8485 5654 50  0000 R CNN
-F 1 "100n" H 8485 5745 50  0000 R CNN
+F 1 "100nF" H 8485 5745 50  0000 R CNN
 F 2 "Capacitor_SMD:C_0805_2012Metric" H 8638 5550 50  0001 C CNN
 F 3 "~" H 8600 5700 50  0001 C CNN

Commit message: repo cleanup and structuring of folders
Parts:
- added J1: ED060SC7, PANASONIC_AXT334124, symbol inkplateclone-rescue:ED060SC7-ED060SC7
- U1: symbol TPS65186:TPS65186 -> inkplateclone-rescue:TPS65186-TPS65186
- U2: symbol ED0970C1:ED097OC1 -> inkplateclone-rescue:ED097OC1-ED0970C1
Connections:
- net 3V3-EINK: now also J1.5 (VDD), J1.7 (VDD)
- net EPD_CKV: now also J1.28 (CKV)
- net EPD_CL: now also J1.9 (XCL)
- net EPD_D0: now also J1.13 (D0)
- net EPD_D1: now also J1.14 (D1)
- net EPD_D2: now also J1.15 (D2)
- net EPD_D3: now also J1.16 (D3)
- net EPD_D4: now also J1.17 (D4)
- net EPD_D5: now also J1.18 (D5)
- net EPD_D6: now also J1.19 (D6)
- net EPD_D7: now also J1.20 (D7)
- net EPD_GMODE: now also J1.26 (MODE1)
- net EPD_LE: now also J1.10 (XLE)
- net EPD_OE: now also J1.11 (XOE)
- net EPD_SPH: now also J1.12 (XSTL)
- net EPD_SPV: now also J1.30 (SPV)
- net GND: now also J1.31 (VSS), J1.32 (BORDER), J1.6 (VSS), J1.8 (VSS)
- net VCOM: now also J1.21 (VCOM), J1.23 (VCOM)
- net VDDH: now also J1.25 (VGG)
- net VEE: now also J1.27 (VEE), J1.29 (VEE)
- net VNEG: now also J1.1 (VNEG), J1.3 (VNEG)
- net VPOS: now also J1.2 (VPOS), J1.4 (VPOS)
Other:
- moved on the sheet: C11, C12, C13, C14, C15, C16, C17, C18, C19, C20, C21, D1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
